File: Hardware/WattMeter.brd (EAGLE design)
At the start: 45.4 x 57.1 mm, 42 parts, among them J1 Molex C136453, J2 AUDIO_JACK_TRRSSMD_RA, Q1 SS8050-G, Q2 SS8050-G, U1 ESP-WROOM-32EU, U2 AMS1117, U3 CH340K, U4 W25Q32FV, U5 ADS1015

Commit message: Защита от скачков по USB
Parts:
- added D1, D2: 5.6V, SparkFun-DiscreteSemi:SOD-323
- added D3: SMF5.0CA, SMF5.0CA:SOD-123FL
- added F1: 6V 0.5A, SparkFun-Fuses:0805
- added U6: AZC099-04S, SamacSys_Parts:SOT95P275X110-6N
Connections:
- new net N$27: F1.1, J1.VBUS1, J5.2
- net +5V: now also D1.C, F1.2, U6.5; no longer J1.VBUS1, J5.2
- net 3.3V: now also D2.C
- net GND: now also D1.A, D2.A, U6.2
- net N$1: now also U6.1
- net N$22: now also D3.P$1
- net N$25: now also D3.P$2
- net N$3: now also U6.3
Routing:
- net N$27: track 0.00 -> 47.7 mm
- net N$3: track 4.30 -> 24.4 mm, vias 0 -> 2
- net N$25: track 32.3 -> 51.1 mm, vias 5 -> 7
- net N$1: track 4.40 -> 18.8 mm, vias 0 -> 2
- net +5V: track 111.1 -> 99.3 mm, vias 0 -> 2
- net GND: track 252.7 -> 260.6 mm, vias 6 -> 8
- net 3.3V: track 207.7 -> 211.8 mm
- net N$22: track 24.9 -> 26.6 mm
