File: Hardware/WattMeter.sch (EAGLE design)
At the start: 42 parts, among them J1 Molex C136453, J2 AUDIO_JACK_TRRSSMD_RA, Q1 SS8050-G, Q2 SS8050-G, U1 ESP-WROOM-32EU, U2 AMS1117, U3 CH340K, U4 W25Q32FV, U5 ADS1015

Commit message: Защита от скачков по USB
Parts:
- added D1, D2: 5.6V, SparkFun-DiscreteSemi:DIODE-ZENER-MMSZ5232BS
- added D3: SMF5.0CA, SMF5.0CA:SMF5.0CA
- added F1: 6V 0.5A, SparkFun-Fuses:PPTC_6V500MA
- added U6: AZC099-04S, SamacSys_Parts:AZC099-04S
Connections:
- new net N$27: F1.1, J1.VBUS, J5.2
- net +5V: now also D1.C, F1.2, U6.VDD; no longer J1.VBUS, J5.2
- net 3.3V: now also D2.C
- net GND: now also D1.A, D2.A, U6.GND
- net N$1: now also U6.IO1
- net N$22: now also D3.1
- net N$25: now also D3.2
- net N$3: now also U6.IO2
Other:
- moved on the sheet: J5
